File: hardware/0.1/chief.sch (KiCad schematic (older format))
At the start: 54 parts, among them J1 USB_C_Receptacle_USB2.0, Q1 DTC123J, Q2 BSS138, SW1 Encoder_MX_RGB, SW10 Encoder_MX_RGB, SW11 MX_RGB, SW12 MX_RGB, SW13 SW_Push, SW2 MX_RGB, SW3 MX_RGB, SW4 Encoder_MX_RGB, SW5 MX_RGB, SW6 MX_RGB, SW7 Encoder_MX_RGB, SW8 MX_RGB, SW9 MX_RGB, U1 AP2112K-3.3, U2 USBLC6-2SC6, U3 STM32F072C8Tx

Commit message: sorry Bing
Parts:
- removed RN5: 5K1, Resistor_SMD:R_Array_Convex_4x0603, symbol chief-rescue:RN-josh-passive
- added R6, R7: 5K1, Resistor_SMD:R_0603_1608Metric, symbol Device:R
Connections:
- net ENC2B_DB: now also U3.26 (PB13); no longer U3.27 (PB14)
- net ENC4A_DB: now also U3.41 (PB5); no longer U3.42 (PB6)
- net ENC4B_DB: now also U3.42 (PB6); no longer U3.46 (PB9)
- net GND: now also R6.1, R7.1
- net SW11: now also U3.43 (PB7); no longer U3.3 (PC14)
- net SW12: now also U3.45 (PB8); no longer U3.10 (PA0)
- net SW5: now also U3.27 (PB14); no longer U3.26 (PB13)
- net SW9: now also U3.46 (PB9); no longer U3.2 (PC13)
- net at J1.A5 (CC1): now also R6.2
- net at J1.B5 (CC2): now also R7.2
Changed lines of the file:
@@
-$EndComp
-$Comp
-L chief-rescue:RN-josh-passive RN5
-U 1 1 604AA3D6
-P 1800 1550
-F 0 "RN5" H 1800 1650 50  0000 C CNN
-F 1 "5K1" H 1800 1550 50  0000 C CNN
-F 2 "Resistor_SMD:R_Array_Convex_4x0603" V 1800 1550 50  0001 C CNN
-F 3 "" V 1800 1550 50  0001 C CNN
-	1    1800 1550
-	1    0    0    -1
-$EndComp
-$Comp
-L chief-rescue:RN-josh-passive RN5
-U 2 1 604AA3DC
-P 1800 1650
-F 0 "RN5" H 1800 1550 50  0000 C CNN
-F 1 "5K1" H 1800 1650 50  0000 C CNN
-F 2 "Resistor_SMD:R_Array_Convex_4x0603" V 1800 1650 50  0001 C CNN
-F 3 "" V 1800 1650 50  0001 C CNN
-	2    1800 1650
-	1    0    0    -1
 $EndComp
 $Comp
@@
 Text Label 5200 5950 2    50   ~ 0
 ENC1A_DB
-Text Label 3000 6150 0    50   ~ 0
+Text Label 3000 5850 0    50   ~ 0
 ENC4B_DB
-Text Label 3000 5850 0    50   ~ 0
+Text Label 3000 5750 0    50   ~ 0
 ENC4A_DB
 Text Label 5200 6650 2    50   ~ 0
@@
 Text Label 5200 6550 2    50   ~ 0
 SW7
-Text Label 3000 4850 0    50   ~ 0
+Text Label 3000 6150 0    50   ~ 0
 SW9
 Text Label 3000 5650 0    50   ~ 0
@@
 	3000 5350 3450 5350
 Wire Wire Line
-	3450 4850 3000 4850
-Text Label 5200 5250 2    50   ~ 0
+	3450 6150 3000 6150
+Text Label 3000 6050 0    50   ~ 0
 SW12
 Wire Wire Line
-	4750 5250 5200 5250
+	3450 6050 3000 6050
 Wire Wire Line
 	5200 5750 4750 5750
@@
 	3000 5650 3450 5650
 Wire Wire Line
-	3000 6150 3450 6150
-Wire Wire Line
 	3000 5850 3450 5850
 Wire Wire Line
-	3450 4950 3000 4950
-Text Label 3000 4950 0    50   ~ 0
+	3000 5750 3450 5750
+Wire Wire Line
+	3450 5950 3000 5950
+Text Label 3000 5950 0    50   ~ 0
 SW11
 Text Label 5200 5850 2    50   ~ 0
@@
 ENC1B_DB
 Wire Wire Line
-	3000 6650 3450 6650
-Wire Wire Line
-	3450 6450 3000 6450
-Text Label 3000 6650 0    50   ~ 0
+	3000 6550 3450 6550
+Text Label 3000 6550 0    50   ~ 0
 ENC2B_DB
-Text Label 3000 6450 0    50   ~ 0
-ENC2A_DB
 $Comp
 L MCU_ST_STM32F0:STM32F072C8Tx U3
@@
 	1    0    0    -1
 $EndComp
-Text Label 3000 6550 0    50   ~ 0
-SW5
-Wire Wire Line
-	3450 6550 3000 6550
 Wire Wire Line
 	3000 5550 3450 5550
@@
 NoConn ~ 3450 4650
 NoConn ~ 3450 5050
-NoConn ~ 3450 5750
-NoConn ~ 3450 5950
-NoConn ~ 3450 6050
 NoConn ~ 3450 6250
 NoConn ~ 3450 6350
@@
 NoConn ~ 4750 5450
 NoConn ~ 4750 5350
+$Comp
+L Device:R R6
+U 1 1 5F016ED5
+P 1800 1550
+F 0 "R6" V 1700 1550 50  0000 C CNN
+F 1 "5K1" V 1800 1550 50  0000 C CNN
+F 2 "Resistor_SMD:R_0603_1608Metric" V 1730 1550 50  0001 C CNN
+F 3 "~" H 1800 1550 50  0001 C CNN
+	1    1800 1550
+	0    1    1    0
+$EndComp
+$Comp
+L Device:R R7
+U 1 1 5F0187ED
+P 1800 1650
+F 0 "R7" V 1900 1650 50  0000 C CNN
+F 1 "5K1" V 1800 1650 50  0000 C CNN
+F 2 "Resistor_SMD:R_0603_1608Metric" V 1730 1650 50  0001 C CNN
+F 3 "~" H 1800 1650 50  0001 C CNN
+	1    1800 1650
+	0    1    1    0
+$EndComp
+Text Label 3000 6450 0    50   ~ 0
+ENC2A_DB
+Wire Wire Line
+	3450 6450 3000 6450
+Wire Wire Line
+	3450 6650 3000 6650
+Text Label 3000 6650 0    50   ~ 0
+SW5
+NoConn ~ 3450 4950
+NoConn ~ 3450 4850
+NoConn ~ 4750 5250
 $EndSCHEMATC

Commit message: moar layout
Parts:
- added D3, D4, D5, D6: WS2812B, LED_SMD:LED_WS2812B_PLCC4_5.0x5.0mm_P3.2mm, symbol LED:WS2812B
- added H5: dan, graphics:danandrews, symbol Mechanical:MountingHole
Connections:
- net +5V: now also D3.1 (VDD), D4.1 (VDD), D5.1 (VDD), D6.1 (VDD)
- net GND: now also D3.3 (VSS), D4.3 (VSS), D5.3 (VSS), D6.3 (VSS)
- net BKLT: now reaches SW12.4 (DO)
- net BKLT: now also D3.4 (DIN)
- new net: D3.2 (DOUT), D4.4 (DIN)
- new net: D4.2 (DOUT), D5.4 (DIN)
- new net: D5.2 (DOUT), D6.4 (DIN)
Other:
- moved on the sheet: C10, C11, C12, C13, C6, C7, C8, C9, RN1A, RN1B, RN1C, RN1D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
